File: hardware/operacake/operacake.sch (KiCad schematic (older format))
At the start: 152 parts, among them J1 CONN_02X20, J2 CONN_02X20, P1 ADDRESS, P20 GPIO, P22 I2S, P28 SD, P9 BASEBAND, U1 MASWSS0129, U10 74LVC1G58, U11 74LVC1G58, U12 74LVC1G58, U13 74LVC1G58, U14 74AHC1G02, U15 74AHC1G02, U16 74LVC1G19, U2 SKY13322, U3 SKY13322, U4 PCA9557, U5 TC7MBL3245CFT, U6 74LVC1G58, U7 74LVC1G58, U8 74AHC1G08, U9 74AHC1G08

Commit message: Changed schematic and PCB to a design that seperates the PA & PB sides. No crossover will be possible with this design.
Parts:
- removed C10, C9: 100nF, gsg-modules:0402, symbol C
- removed C17, C18: 33pF, gsg-modules:0402, symbol C
- removed U1: MASWSS0129, gsg-modules:QFN12-3, symbol MASWSS0129
Connections:
- wire segments 408 -> 390
- no-connect marks 137 -> 138
Changed lines of the file:
@@
 $EndComp
 $Comp
-L MASWSS0129 U1
-U 1 1 57ED7D40
-P 5900 5450
-F 0 "U1" H 5900 5500 40  0000 C CNN
-F 1 "MASWSS0129" H 5900 5400 40  0000 C CNN
-F 2 "gsg-modules:QFN12-3" H 5900 5450 60  0001 C CNN
-F 3 "" H 5900 5450 60  0000 C CNN
-F 4 "M/A-Com" H 5900 5450 60  0001 C CNN "Manufacturer"
-F 5 "MASWSS0129TR-3000" H 5900 5450 60  0001 C CNN "Part Number"
-F 6 "DPDT LEAD FREE SWITCH DC - 6GHZ" H 5900 5450 60  0001 C CNN "Description"
-	1    5900 5450
-	-1   0    0    1
-$EndComp
-$Comp
 L GND #PWR020
 U 1 1 57ED8360
@@
 $EndComp
 $Comp
-L GND #PWR022
-U 1 1 57EDA016
-P 5900 6050
-F 0 "#PWR022" H 5900 5800 50  0001 C CNN
-F 1 "GND" H 5900 5900 50  0000 C CNN
-F 2 "" H 5900 6050 60  0000 C CNN
-F 3 "" H 5900 6050 60  0000 C CNN
-	1    5900 6050
-	1    0    0    -1
-$EndComp
-$Comp
-L GND #PWR023
-U 1 1 57EDA14E
-P 6500 5800
-F 0 "#PWR023" H 6500 5550 50  0001 C CNN
-F 1 "GND" H 6500 5650 50  0000 C CNN
-F 2 "" H 6500 5800 60  0000 C CNN
-F 3 "" H 6500 5800 60  0000 C CNN
-	1    6500 5800
-	1    0    0    -1
-$EndComp
-$Comp
-L GND #PWR024
-U 1 1 57EDA784
-P 5300 5650
-F 0 "#PWR024" H 5300 5400 50  0001 C CNN
-F 1 "GND" H 5300 5500 50  0000 C CNN
-F 2 "" H 5300 5650 60  0000 C CNN
-F 3 "" H 5300 5650 60  0000 C CNN
-	1    5300 5650
-	1    0    0    -1
-$EndComp
-$Comp
-L GND #PWR025
-U 1 1 57EDABAF
-P 5900 4850
-F 0 "#PWR025" H 5900 4600 50  0001 C CNN
-F 1 "GND" H 5900 4700 50  0000 C CNN
-F 2 "" H 5900 4850 60  0000 C CNN
-F 3 "" H 5900 4850 60  0000 C CNN
-	1    5900 4850
-	-1   0    0    1
-$EndComp
-$Comp
-L C C9
-U 1 1 57EDB85B
-P 4950 4600
-F 0 "C9" H 4975 4700 50  0000 L CNN
-F 1 "100nF" H 4975 4500 50  0000 L CNN
-F 2 "gsg-modules:0402" H 4988 4450 30  0001 C CNN
-F 3 "" H 4950 4600 60  0000 C CNN
-F 4 "Murata" H 4950 4600 60  0001 C CNN "Manufacturer"
-F 5 "GRM155R61A104KA01D" H 4950 4600 60  0001 C CNN "Part Number"
-F 6 "CAP CER 0.1UF 10V 10% X5R 0402" H 4950 4600 60  0001 C CNN "Description"
-	1    4950 4600
-	0    1    1    0
-$EndComp
-$Comp
-L C C10
-U 1 1 57EDC2D6
-P 6900 4600
-F 0 "C10" H 6925 4700 50  0000 L CNN
-F 1 "100nF" H 6925 4500 50  0000 L CNN
-F 2 "gsg-modules:0402" H 6938 4450 30  0001 C CNN
-F 3 "" H 6900 4600 60  0000 C CNN
-F 4 "Murata" H 6900 4600 60  0001 C CNN "Manufacturer"
-F 5 "GRM155R61A104KA01D" H 6900 4600 60  0001 C CNN "Part Number"
-F 6 "CAP CER 0.1UF 10V 10% X5R 0402" H 6900 4600 60  0001 C CNN "Description"
-	1    6900 4600
-	0    1    1    0
-$EndComp
-$Comp
 L GSG-RF-CONN PA1
 U 1 1 57EF0A3B
@@
 	0    -1   -1   0
 $EndComp
-Text Label 4900 5350 0    40   ~ 0
-U1VC2
-Text Label 6900 5350 2    40   ~ 0
-U1VC1
 Text Label 3200 5050 1    40   ~ 0
 U2V4
@@
 Text Label 14100 5300 2    40   ~ 0
 U2V1
-Text Label 16150 7850 2    40   ~ 0
-U1VC1
-Text Label 16150 7650 2    40   ~ 0
-U1VC2
 Text Label 16150 6100 2    40   ~ 0
 U3V4
@@
 $EndComp
 $Comp
-L C C17
-U 1 1 59504505
-P 5250 5050
-F 0 "C17" H 5275 5150 50  0000 L CNN
-F 1 "33pF" H 5275 4950 50  0000 L CNN
-F 2 "gsg-modules:0402" H 5288 4900 50  0001 C CNN
-F 3 "" H 5250 5050 50  0000 C CNN
-F 4 "Murata" H 5250 5050 60  0001 C CNN "Manufacturer"
-F 5 "GRM1555C1H330JA01D" H 5250 5050 60  0001 C CNN "Part Number"
-F 6 "CAP CER 33PF 50V 5% NP0 0402" H 5250 5050 60  0001 C CNN "Description"
-	1    5250 5050
-	1    0    0    -1
-$EndComp
-$Comp
-L GND #PWR089
-U 1 1 59504628
-P 5250 4900
-F 0 "#PWR089" H 5250 4650 50  0001 C CNN
-F 1 "GND" H 5250 4750 50  0000 C CNN
-F 2 "" H 5250 4900 50  0000 C CNN
-F 3 "" H 5250 4900 50  0000 C CNN
-	1    5250 4900
-	-1   0    0    1
-$EndComp
-$Comp
-L GND #PWR090
-U 1 1 5950496C
-P 6550 4900
-F 0 "#PWR090" H 6550 4650 50  0001 C CNN
-F 1 "GND" H 6550 4750 50  0000 C CNN
-F 2 "" H 6550 4900 50  0000 C CNN
-F 3 "" H 6550 4900 50  0000 C CNN
-	1    6550 4900
-	-1   0    0    1
-$EndComp
-$Comp
-L C C18
-U 1 1 59504CB0
-P 6550 5050
-F 0 "C18" H 6575 5150 50  0000 L CNN
-F 1 "33pF" H 6575 4950 50  0000 L CNN
-F 2 "gsg-modules:0402" H 6588 4900 50  0001 C CNN
-F 3 "" H 6550 5050 50  0000 C CNN
-F 4 "Murata" H 6550 5050 60  0001 C CNN "Manufacturer"
-F 5 "GRM1555C1H330JA01D" H 6550 5050 60  0001 C CNN "Part Number"
-F 6 "CAP CER 33PF 50V 5% NP0 0402" H 6550 5050 60  0001 C CNN "Description"
-	1    6550 5050
-	1    0    0    -1
-$EndComp
-$Comp
 L C C13
 U 1 1 5950597B
@@
 	3200 4400 3200 5050
 Wire Wire Line
-	4900 5350 5400 5350
-Wire Wire Line
-	6400 5350 6900 5350
-Wire Wire Line
 	16150 6100 15950 6100
 Wire Wire Line
@@
 	15950 3900 16150 3900
 Wire Wire Line
-	16150 7850 15950 7850
-Wire Wire Line
-	15950 7650 16150 7650
-Wire Wire Line
 	14100 6100 13900 6100
 Wire Wire Line
@@
 	4900 7350 5000 7350
 Wire Wire Line
-	3100 4600 4800 4600
-Wire Wire Line
-	8200 4600 7050 4600
-Wire Wire Line
-	5800 4600 5100 4600
-Wire Wire Line
-	6000 4600 6750 4600
-Wire Wire Line
-	5900 4850 5900 4950
+	3100 4600 5800 4600
 Wire Wire Line
-	5900 5950 5900 6050
-Connection ~ 5300 5550
+	6000 4600 8200 4600
 Wire Wire Line
-	5300 5550 5400 5550
+	6000 4600 6000 7350
 Wire Wire Line
-	5300 5450 5300 5650
+	5800 4600 5800 6200
 Wire Wire Line
-	5400 5450 5300 5450
-Connection ~ 6500 5550
+	5800 6200 5300 6200
 Wire Wire Line
-	6400 5550 6500 5550
-Connection ~ 6500 5700
-Wire Wire Line
-	6500 5700 6400 5700
-Wire Wire Line
-	6500 5450 6500 5800
-Wire Wire Line
-	6400 5450 6500 5450
-Wire Wire Line
-	6000 7350 6000 5950
-Wire Wire Line
-	5800 6200 5800 5950
-Wire Wire Line
-	5300 6200 5800 6200
-Wire Wire Line
-	6000 4600 6000 4950
-Wire Wire Line
-	8200 4400 8200 4600
-Wire Wire Line
-	5800 4600 5800 4950
+	8200 4600 8200 4400
 Wire Wire Line
 	3100 4400 3100 4600
@@
 Connection ~ 5550 7350
 Wire Wire Line
-	5300 7350 6000 7350
+	6000 7350 5300 7350
 Wire Wire Line
 	4600 7750 4600 7850
@@
 Connection ~ 3200 3250
 Wire Wire Line
-	6550 5200 6550 5350
-Connection ~ 6550 5350
-Wire Wire Line
-	5250 5200 5250 5350
-Connection ~ 5250 5350
-Wire Wire Line
 	3300 4750 3200 4750
 Connection ~ 3200 4750
@@
 Wire Wire Line
 	15950 5900 16300 5900
+Text Label 16150 7850 2    40   ~ 0
+U1VC1
+Wire Wire Line
+	16150 7850 15950 7850
+NoConn ~ 15950 7650
 $EndSCHEMATC
